File: PCB/totem_compact/totem_compact.kicad_pcb (KiCad board)
At the start: 2 copper layers, 130.9 x 95.6 mm, 43 parts, among them U1 xiao-ble

Commit message: Update PCB
Parts:
- RST: renamed from LSW1; footprint Button_Switch_THT:SW_PUSH_6mm -> TOTEMlib:Diode_SOD123
- moved RST 58.2 mm to (159.0, 116.5), turned to -90 degrees
- moved BAT+1L1 2.92 mm to (94.0, 103.0)
- moved BAT-1L1 2.92 mm to (89.5, 103.0)
Routing:
- net COL0_L: track 0.00 -> 223.7 mm, vias 0 -> 7
- net COL2_L: track 0.00 -> 196.2 mm, vias 0 -> 2
- net COL1_L: track 0.00 -> 189.8 mm, vias 0 -> 3
- net COL3_L: track 0.00 -> 169.4 mm
- net Net-(DL1-A): track 0.00 -> 157.6 mm, vias 0 -> 5
- net COL4_L: track 0.00 -> 153.0 mm
- net BAT+L: track 0.00 -> 151.1 mm, vias 0 -> 7
- net Net-(DL6-A): track 0.00 -> 132.3 mm
- net Net-(DL16-A): track 61.8 -> 192.9 mm, vias 0 -> 3
- net Net-(DL11-A): track 0.00 -> 114.2 mm, vias 0 -> 5
- net Net-(DL2-A): track 35.4 -> 143.3 mm
- net Net-(DL7-A): track 32.2 -> 122.7 mm
- net Net-(DL3-A): track 49.5 -> 134.6 mm
- net Net-(DL17-A): track 57.4 -> 127.9 mm, vias 0 -> 1
- net Net-(DL8-A): track 46.0 -> 113.1 mm
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- added copper zone on B.Cu, net GND_L
- added copper zone on F.Cu, net GND_L
