File: PCB/totem_compact/totem_compact.kicad_sch (KiCad schematic)
At the start: 86 parts, among them U1 xiao-ble, U2 xiao-ble

Commit message: Update PCB
Parts:
- LSW1: footprint Button_Switch_THT:SW_PUSH_6mm -> TOTEMlib:Diode_SOD123
Changed lines of the file:
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@@
 			)
 		)
-		(property "Footprint" "Button_Switch_THT:SW_PUSH_6mm"
+		(property "Footprint" "TOTEMlib:Diode_SOD123"
 			(at 116.84 64.77 0)
 			(effects
